File: pump_hw/pump_hw.kicad_sch (KiCad schematic)
At the start: 0 parts

Commit message: power switching thoughts
Parts:
- added U1: ATSAMD21G18A-A, Package_QFP:TQFP-48_7x7mm_P0.5mm, symbol MCU_Microchip_SAMD:ATSAMD21G18A-A
Connections:
- new net: U1.18 (GND), U1.35 (GND), U1.42 (GND)
Changed lines of the file:
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@@
 	(generator_version "9.0")
 	(paper "A4")
+	(symbol
+		(lib_id "MCU_Microchip_SAMD:ATSAMD21G18A-A")
+		(at 237.49 81.28 0)
+		(unit 1)
+		(exclude_from_sim no)
+		(in_bom yes)
+		(on_board yes)
+		(dnp no)
+		(fields_autoplaced yes)
+		(property "Reference" "U1"
+			(at 242.1733 129.54 0)
+			(effects
+				(font
+					(size 1.27 1.27)
+				)
+				(justify left)
+			)
+		)
+		(property "Value" "ATSAMD21G18A-A"
+			(at 242.1733 132.08 0)
+			(effects
+				(font
+					(size 1.27 1.27)
+				)
+				(justify left)
+			)
+		)
+		(property "Footprint" "Package_QFP:TQFP-48_7x7mm_P0.5mm"
+			(at 260.35 128.27 0)
+			(effects
+				(font
+					(size 1.27 1.27)
+				)
+				(hide yes)
+			)
+		)
+		(property "Datasheet" "http://ww1.microchip.com/downloads/en/DeviceDoc/SAM_D21_DA1_Family_Data%20Sheet_DS40001882E.pdf"
+			(at 237.49 55.88 0)
+			(effects
+				(font
+					(size 1.27 1.27)
+				)
+				(hide yes)
+			)
+		)
+		(property "Description" "SAM D21 Microchip SMART ARM-based Flash MCU, 48Mhz, 256K Flash, 32K SRAM, TQFP-48"
+			(at 237.49 81.28 0)
+			(effects
+				(font
+					(size 1.27 1.27)
+				)
+				(hide yes)
+			)
+		)
+		(pin "1"
+		)
+		(pin "29"
+		)
+		(pin "33"
+		)
+		(pin "39"
+		)
+		(pin "45"
+		)
+		(pin "22"
+		)
+		(pin "4"
+		)
+		(pin "10"
+		)
+		(pin "13"
+		)
+		(pin "12"
+		)
+		(pin "2"
+		)
+		(pin "9"
+		)
+		(pin "11"
+		)
+		(pin "3"
+		)
+		(pin "25"
+		)
+		(pin "21"
+		)
+		(pin "23"
+		)
+		(pin "26"
+		)
+		(pin "28"
+		)
+		(pin "15"
+		)
+		(pin "30"
+		)
+		(pin "31"
+		)
+		(pin "16"
+		)
+		(pin "24"
+		)
+		(pin "27"
+		)
+		(pin "14"
+		)
+		(pin "32"
+		)
+		(pin "34"
+		)
+		(pin "41"
+		)
+		(pin "8"
+		)
+		(pin "46"
+		)
+		(pin "20"
+		)
+		(pin "40"
+		)
+		(pin "36"
+		)
+		(pin "5"
+		)
+		(pin "7"
+		)
+		(pin "48"
+		)
+		(pin "37"
+		)
+		(pin "43"
+		)
+		(pin "44"
+		)
+		(pin "42"
+		)
+		(pin "35"
+		)
+		(pin "17"
+		)
+		(pin "47"
+		)
+		(pin "19"
+		)
+		(pin "18"
+		)
+		(pin "6"
+		)
+		(pin "38"
+		)
+		(instances
+			(project ""
+				(path "/c52da85b-ae68-4cb2-bfa9-3df305c88992"
+					(reference "U1")
+					(unit 1)
+				)
+			)
+		)
+	)
 	(sheet_instances
 		(path "/"
