File: pump/pump.kicad_sch (KiCad schematic)
At the start: 1 part, among them U3 40PC015G

Commit message: added avr64da64 as mcu and basic decoupling on power pins
Other:
- added sheet Mcu (mcu.kicad_sch)
Changed lines of the file:
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@@
+		)
+	)
+	(sheet
+		(at 115.57 121.92)
+		(size 16.51 15.24)
+		(exclude_from_sim no)
+		(in_bom yes)
+		(on_board yes)
+		(dnp no)
+		(fields_autoplaced yes)
+		(stroke
+			(width 0.1524)
+			(type solid)
+		)
+		(fill
+			(color 0 0 0 0.0000)
+		)
+		(property "Sheetname" "Mcu"
+			(at 115.57 121.2084 0)
+			(effects
+				(font
+					(size 1.27 1.27)
+				)
+				(justify left bottom)
+			)
+		)
+		(property "Sheetfile" "mcu.kicad_sch"
+			(at 115.57 137.7446 0)
+			(effects
+				(font
+					(size 1.27 1.27)
+				)
+				(justify left top)
+			)
+		)
+		(instances
+			(project "pump"
+				(path "/e0be0fc6-35a9-4dbe-8638-3e88dcb86763"
+					(page "3")
+				)
+			)
 		)
 	)

Commit message: finished control relays schematic and footprints
Parts:
- U3: footprint (none) -> TerminalBlock:TerminalBlock_MaiXu_MX126-5.0-06P_1x06_P5.00mm
Changed lines of the file:
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@@
 			)
 		)
-		(property "Footprint" ""
+		(property "Footprint" "TerminalBlock:TerminalBlock_MaiXu_MX126-5.0-06P_1x06_P5.00mm"
 			(at 196.85 151.13 0)
 			(effects

Commit message: time to go
Parts:
- removed U3: 40PC015G, TerminalBlock:TerminalBlock_MaiXu_MX126-5.0-06P_1x06_P5.00mm, symbol Sensor_Pressure:40PC015G
- added J2: Conn_01x04_Pin, symbol Connector:Conn_01x04_Pin
- added J3: Conn_01x03_Pin, symbol Connector:Conn_01x03_Pin
- added PS1: IRM-20-12, Converter_ACDC:Converter_ACDC_MeanWell_IRM-20-xx_THT, symbol Converter_ACDC:IRM-20-12
- added PS2: RAC20-12SK, Converter_ACDC:Converter_ACDC_Recom_RAC20-xxSK_THT, symbol Converter_ACDC:RAC20-12SK
Connections:
- net +5V: now also J2.2 (Pin_2), J3.2 (Pin_2)
- net GND: now also J2.1 (Pin_1), J3.1 (Pin_1)
- net P_SENSOR_READING: now also J3.3 (Pin_3)
- new net LTE_RX: J2.3 (Pin_3)
- new net LTE_TX: J2.4 (Pin_4)
Other:
- note removed: "10mA @5V"
